File: Electrical/VolleyBot.kicad_pcb (KiCad board)
At the start: 2 copper layers, 95.2 x 57.5 mm, 66 parts, among them J1 Conn_01x04_Pin, J2 Conn_01x04_Pin, J3 Conn_01x02_Pin, J4 Conn_01x04_Socket, J5 Conn_01x02_Socket, J6 Conn_01x02_Socket, J7 Conn_01x02_Socket, SW1 SW_SPDT, U1 STM32F411CEU6, U2 DRV8833PWP, U3 DRV8833PWP, U4 AP62300TWU, U5 AP62300TWU, Y1 16MHz

Commit message: routed pcb
Parts:
- J3: footprint TerminalBlock:TerminalBlock_MaiXu_MX126-5.0-02P_1x02_P5.00mm -> Rocketry_Manual:Screw_Terminal_2_Pins
- moved J5 33.4 mm to (84.8, 106.6), turned to 0 degrees
- moved J7 31.6 mm to (101.8, 106.6), turned to 0 degrees
- moved J6 30.2 mm to (93.2, 106.6), turned to 0 degrees
- moved D2 19.9 mm to (121.2, 114.2)
- moved R7 15.9 mm to (119.8, 114.8)
- moved R1 13.5 mm to (105.3, 71.5)
- moved H4 10.1 mm to (77.5, 68.2)
- moved H2 9.71 mm to (77.5, 112.2)
- moved R2 9.28 mm to (144.2, 78.2)
- moved R3 9.28 mm to (144.2, 83.8)
- moved USB2 9.28 mm to (148.4, 81.0)
- moved H1 6.73 mm to (149.5, 68.2)
- moved H3 6.09 mm to (149.5, 112.2)
- moved H5 4.25 mm to (84.5, 69.5)
- moved H6 4.25 mm to (142.5, 69.5)
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Connections:
- C18 pad 1: /VBATT -> +BATT
- C21 pad 1: /VBATT -> +BATT
- U2 pad 12: /VBATT -> +BATT
- U3 pad 12: /VBATT -> +BATT
Routing:
- net +3.3V: track 63.1 -> 174.1 mm, vias 3 -> 18
- net +BATT: track 0.00 -> 73.0 mm, vias 0 -> 3
- net +5V: track 0.00 -> 21.8 mm, vias 0 -> 2
- net Net-(SW1-B): track 20.9 -> 5.65 mm
- net /BOOT0: track 3.94 -> 18.5 mm
- net -BATT: track 64.7 -> 71.2 mm, vias 7 -> 27
- net /USB_D-: track 33.1 -> 26.6 mm
- net /USB_D+: track 33.1 -> 26.6 mm
- net VBUS: track 37.0 -> 42.1 mm
- net /USART1_RX: track 9.02 -> 14.0 mm
- net Net-(J5-Pin_1): track 25.6 -> 29.9 mm
- net /USART1_TX: track 6.99 -> 11.2 mm
- net Net-(J4-Pin_2): track 11.2 -> 7.66 mm
- net Net-(J4-Pin_3): track 12.0 -> 8.49 mm
- net /SWDIO: track 17.0 -> 13.5 mm
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- added copper zone on F.Cu, net +3.3V
- added copper zone on F.Cu, net +5V
- added copper zone on F.Cu, net +BATT
- added copper zone on F.Cu, net -BATT
- added copper zone on F.Cu, net /BST1
- added copper zone on F.Cu, net /BST2
- added copper zone on F.Cu, net /FB1
- added copper zone on F.Cu, net /FB2
- added copper zone on F.Cu, net /SW1
- added copper zone on F.Cu, net /SW2
Other:
- board size 95.2 x 57.5 mm -> 80 x 52 mm
- board text added: "GYRO CONN"
- board text added: "MOTOR 1"
- board text added: "MOTOR 2"
- board text added: "MOTOR 3"
- board text added: "MOTOR DRIVER 1"
- board text added: "MOTOR DRIVER 2"
- board text added: "POWER LED"
- board text added: "RPI ZERO 2 W CONN"
- board text added: "SERIAL DEBUG"
- board text added: "VolleyBot"

Commit message: pcb made
Parts:
- added D4: LED, LED_SMD:LED_0603_1608Metric, F.Cu at (131.0, 113.5)
- added D5: LED, LED_SMD:LED_0603_1608Metric, F.Cu at (123.8, 113.5)
- added G***: LOGO, LOGO, F.Cu at (92.7, 81.0)
- added Q1: AO3401A, Rocketry_Easyeda:SOT-23_L2.9-W1.3-P1.90-LS2.4-BR, F.Cu at (132.5, 97.2)
- added Q2: AO3401A, Rocketry_Easyeda:SOT-23_L2.9-W1.3-P1.90-LS2.4-BR, F.Cu at (107.2, 106.5)
- added R13: 220R, Resistor_SMD:R_0402_1005Metric, F.Cu at (130.5, 112.0)
- added R19: 10K, Resistor_SMD:R_0402_1005Metric, F.Cu at (106.8, 109.0)
- added R20: 220R, Resistor_SMD:R_0402_1005Metric, F.Cu at (124.2, 112.0)
- added R4: 10K, Resistor_SMD:R_0402_1005Metric, F.Cu at (131.2, 101.0)
- added SW2: SW_SPDT, Button_Switch_SMD:SW_SPDT_PCM12, F.Cu at (139.8, 113.8)
- added SW3: SW_SPDT, Button_Switch_SMD:SW_SPDT_PCM12, F.Cu at (109.8, 113.8)
- J3: value Conn_01x02_Pin -> Conn_01x02_Socket; footprint Rocketry_Manual:Screw_Terminal_2_Pins -> Connector_AMASS:AMASS_XT60PW-F_1x02_P7.20mm_Horizontal
- R5: value 6K8 -> 15K
- moved J5 31.1 mm to (82.9, 75.5), turned to -90 degrees
- moved J6 24.8 mm to (82.9, 84.0), turned to -90 degrees
- moved J3 23.8 mm to (91.7, 100.8)
- moved J7 20.5 mm to (82.9, 98.5), turned to -90 degrees
- moved D2 4.35 mm to (117.0, 113.5), turned to 180 degrees
- moved R7 3.62 mm to (117.4, 112.0), turned to 0 degrees
- moved D3 3.35 mm to (121.0, 94.2)
- moved D1 1.56 mm to (131.8, 110.0)
- moved C20 1.00 mm to (101.6, 93.2)
- moved U3 0.81 mm to (96.4, 94.2)
- moved C19 0.75 mm to (101.7, 95.5)
- moved SW1 0.75 mm to (103.0, 66.8)
- moved C16 0.67 mm to (101.7, 86.8)
- moved C17 0.67 mm to (101.7, 88.8)
- moved C21 0.67 mm to (104.4, 87.8)
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Connections:
- net Net-(J4-Pin_2) renamed /I2C1_SCL
- net Net-(J4-Pin_3) renamed /I2C1_SDA
- C12 pad 1: +BATT -> /BATT+_IN
- C18 pad 1: +BATT -> /BATT+_IN
- C21 pad 1: +BATT -> /BATT+_IN
- C23 pad 1: +BATT -> /BATT+_IN
- D1 pad 1: +BATT -> /BATT+_IN
- J1 pad 4: +5V -> /PI_POWER
- R5 pad 1: +BATT -> /BATT+_IN
- U1 pad 29: unconnected-(U1-PA8-Pad29) -> /I2C3_SCL
- U1 pad 40: unconnected-(U1-PB4-Pad40) -> /I2C3_SDA
- U2 pad 12: +BATT -> /BATT+_IN
- U3 pad 12: +BATT -> /BATT+_IN
- U4 pad 3: +BATT -> /BATT+_IN
- U5 pad 3: +BATT -> /BATT+_IN
Routing:
- net /BATT+_IN: track 0.00 -> 70.1 mm, vias 0 -> 3
- net +BATT: track 73.0 -> 20.8 mm, vias 3 -> 0
- net /PI_POWER: track 0.00 -> 21.6 mm, vias 0 -> 2
- net Net-(SW2-A): track 0.00 -> 13.8 mm, vias 0 -> 2
- net Net-(J5-Pin_1): track 29.9 -> 17.1 mm
- net Net-(J6-Pin_1): track 23.6 -> 12.3 mm
- net Net-(J6-Pin_2): track 21.7 -> 11.8 mm
- net Net-(J7-Pin_1): track 22.4 -> 13.0 mm
- net Net-(J5-Pin_2): track 23.9 -> 16.3 mm
- net Net-(J7-Pin_2): track 21.2 -> 13.7 mm
- net VBUS: track 42.1 -> 46.8 mm
- net Net-(D3-A): track 6.96 -> 10.6 mm
- net Net-(SW3-A): track 0.00 -> 3.17 mm
- net -BATT: track 71.2 -> 73.4 mm
- net Net-(SW1-B): track 5.65 -> 3.78 mm
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- added copper zone on F.Cu, net /BATT+_IN
- removed copper zone on F.Cu, net +BATT
Other:
- board text added: "BATT"
- board text added: "BATT SWITCH"
- board text added: "BOOT MODE SWITCH"
- board text added: "IMU CONN"
- board text added: "POWER"
- board text added: "RPI POWER"
- board text added: "RPI POWER SWITCH"
- board text added: "RPI ZERO 2W CONN"
- board text added: "STM LED"
- board text removed: "+"
- board text removed: "-"
- board text removed: "GYRO CONN"
- board text removed: "MOTOR DRIVER 1"
- board text removed: "MOTOR DRIVER 2"
- board text removed: "POWER LED"
- board text removed: "RPI ZERO 2 W CONN"

Commit message: correction of manufacturing files
Parts:
- removed R19: 10K, Resistor_SMD:R_0402_1005Metric
- added R21: 10K, Resistor_SMD:R_0402_1005Metric, F.Cu at (108.8, 108.0)
- C1, C12, C18, C21, C23: value 10u -> 10uF
- C10, C9: value 10p -> 10pF
- C14, C15, C25, C26: value 22u -> 22uF
- C17, C19: value 10n -> 10nF
- C2, C22, C24, C3, C4, C8: value 100n -> 100nF
- C5: value 10n -> 100nF
- C6, C7: value 1u -> 1uF
- FB1: value 120R -> 600R
- R11: footprint Resistor_SMD:R_0402_1005Metric -> Resistor_SMD:R_0603_1608Metric
- moved R4 11.9 mm to (140.0, 109.0), turned to 180 degrees
- moved Q2 1.41 mm to (106.2, 105.5), turned to 180 degrees
- moved Q1 1.00 mm to (133.5, 97.2)
- moved R11 0.55 mm to (131.5, 107.0)
Connections:
- Q1 pad 1: +5V -> Net-(Q1-G)
- Q2 pad 1: +BATT -> Net-(Q2-G)
- R4 pad 1: Net-(SW2-A) -> Net-(SW2-B)
- R4 pad 2: +5V -> Net-(Q1-G)
- SW2 pad 1: Net-(SW2-A) -> +5V
- SW2 pad 2: -BATT -> Net-(SW2-B)
- SW2 pad 3: unconnected-(SW2-C-Pad3) -> -BATT
- SW3 pad 1: Net-(SW3-A) -> +BATT
- SW3 pad 2: -BATT -> Net-(SW3-B)
- SW3 pad 3: unconnected-(SW3-C-Pad3) -> -BATT
Routing:
- net +5V: track 21.1 -> 40.1 mm, vias 2 -> 4
- net Net-(Q1-G): track 0.00 -> 15.7 mm, vias 0 -> 2
- net Net-(SW2-A): track 13.8 -> 0.00 mm, vias 2 -> 0
- net Net-(SW3-B): track 0.00 -> 4.83 mm
- net Net-(Q2-G): track 0.00 -> 4.75 mm
- net Net-(SW2-B): track 0.00 -> 3.35 mm
- net Net-(SW3-A): track 3.17 -> 0.00 mm
- net +BATT: track 20.8 -> 22.7 mm

Commit message: schem done
Parts:
- removed R20: 220R, Resistor_SMD:R_0402_1005Metric
- added BUZZER1: FUET-8530H-3.6V, Rocketry_Easyeda:BUZ-SMD_4P-L8.5-W8.5_FUET-8530-05, F.Cu at (118.0, 69.2)
- added C27: 10uF, Capacitor_SMD:C_0603_1608Metric, F.Cu at (114.2, 90.6)
- added C28: 10uF, Capacitor_SMD:C_0603_1608Metric, F.Cu at (115.8, 90.6)
- added C29: 22uF, Capacitor_SMD:C_0805_2012Metric, F.Cu at (117.5, 90.9)
- added C30: 22uF, Capacitor_SMD:C_0805_2012Metric, F.Cu at (119.7, 90.9)
- added C31: 100nF, Capacitor_SMD:C_0402_1005Metric, F.Cu at (110.6, 94.8)
- added C32: 10uF, Capacitor_SMD:C_0603_1608Metric, F.Cu at (113.8, 94.7)
- added C33: 10uF, Capacitor_SMD:C_0603_1608Metric, F.Cu at (107.7, 94.7)
- added C34: 100nF, Capacitor_SMD:C_0402_1005Metric, F.Cu at (108.8, 104.5)
- added C35: 100nF, Capacitor_SMD:C_0402_1005Metric, F.Cu at (111.5, 104.5)
- added D10: SS34_C8678, Rocketry_Easyeda:SMA_L4.3-W2.6-LS5.2-RD, F.Cu at (102.6, 87.7)
- added D12: SS34_C8678, Rocketry_Easyeda:SMA_L4.3-W2.6-LS5.2-RD, F.Cu at (123.1, 107.7)
- added D6: LED, LED_SMD:LED_0603_1608Metric, F.Cu at (193.8, 81.3)
- added D7: 1N5819WS, Diode_SMD:D_SOD-323, F.Cu at (202.1, 100.6)
- added D8: 1N5819WS, Diode_SMD:D_SOD-323, F.Cu at (202.1, 103.6)
- added D9: SS34_C8678, Rocketry_Easyeda:SMA_L4.3-W2.6-LS5.2-RD, F.Cu at (102.6, 94.5)
- added L4: FNR6045S2R2MT, Rocketry_Easyeda:IND-SMD_L6.0-W6.0_FNR60XXS, F.Cu at (110.8, 99.8)
- added Q3: AO3400A, Rocketry_Easyeda:SOT-23-3_L2.9-W1.3-P1.90-LS2.4-BR, F.Cu at (130.6, 111.5)
- added Q4: SS8050, Package_TO_SOT_SMD:SOT-23, F.Cu at (122.3, 77.9)
- added Q5: AO3401A, Rocketry_Easyeda:SOT-23_L2.9-W1.3-P1.90-LS2.4-BR, F.Cu at (130.5, 114.8)
- added R14: 5K1, Resistor_SMD:R_0402_1005Metric, F.Cu at (115.2, 94.8)
- added R15: 1K, Resistor_SMD:R_0402_1005Metric, F.Cu at (192.7, 102.1)
- added R16: 91K, Resistor_SMD:R_0603_1608Metric, F.Cu at (181.8, 93.3)
- added R17: 120K, Resistor_SMD:R_0603_1608Metric, F.Cu at (181.8, 95.8)
- added R18: 51K, Resistor_SMD:R_0603_1608Metric, F.Cu at (181.8, 98.3)
- added R19: 100R, Resistor_SMD:R_1206_3216Metric, F.Cu at (116.0, 100.5)
- added R22: 680R, Resistor_SMD:R_0402_1005Metric, F.Cu at (195.6, 100.1)
- added R23: 10K, Resistor_SMD:R_0402_1005Metric, F.Cu at (195.6, 102.1)
- added R24: 5K1, Resistor_SMD:R_0402_1005Metric, F.Cu at (195.6, 104.1)
- added R25: 100K, Resistor_SMD:R_0603_1608Metric, F.Cu at (186.6, 105.6)
- added R26: 10K, Resistor_SMD:R_0402_1005Metric, F.Cu at (198.5, 100.1)
- added R27: 1K, Resistor_SMD:R_0402_1005Metric, F.Cu at (198.5, 102.1)
- added R28: 1K, Resistor_SMD:R_0402_1005Metric, F.Cu at (198.5, 104.1)
- added U6: LSM6DSL, Package_LGA:LGA-14_3x2.5mm_P0.5mm_LayoutBorder3x4y, F.Cu at (107.3, 67.5)
- added U7: IP2326, Rocketry_Easyeda:VQFN-24_L4.0-W4.0-P0.50-BL-EP2.5, F.Cu at (110.8, 91.7)
- C16: value 2.2uF -> 10uF; footprint Capacitor_SMD:C_0402_1005Metric -> Capacitor_SMD:C_0603_1608Metric
- C17: value 10nF -> 100nF
- C18, C21: value 10uF -> 100nF; footprint Capacitor_SMD:C_0603_1608Metric -> Capacitor_SMD:C_0402_1005Metric
- C19: value 10nF -> 10uF; footprint Capacitor_SMD:C_0402_1005Metric -> Capacitor_SMD:C_0603_1608Metric
- C20: value 2.2uF -> 100nF
- C6: value 1uF -> 10uF; footprint Capacitor_SMD:C_0402_1005Metric -> Capacitor_SMD:C_0603_1608Metric
- C7: value 1uF -> 10uF; footprint Capacitor_SMD:C_0402_1005Metric -> Capacitor_SMD:C_0805_2012Metric
- C8: value 100nF -> 10uF; footprint Capacitor_SMD:C_0402_1005Metric -> Capacitor_SMD:C_0805_2012Metric
- D1: value 1N5819WS -> SS34_C8678; footprint Diode_SMD:D_SOD-323 -> Rocketry_Easyeda:SMA_L4.3-W2.6-LS5.2-RD
- FB1: value 600R -> C14709
- J2: value Conn_01x04_Pin -> Conn_01x05_Socket; footprint Connector_PinHeader_2.54mm:PinHeader_1x04_P2.54mm_Horizontal -> Connector_JST:JST_XH_S5B-XH-A_1x05_P2.50mm_Horizontal
- J4: value Conn_01x04_Socket -> Conn_01x03_Socket; footprint Connector_JST:JST_XH_S4B-XH-A_1x04_P2.50mm_Horizontal -> Connector_JST:JST_XH_S3B-XH-A_1x03_P2.50mm_Horizontal
- R11: value 56K -> 63.4K
- R12, R13: value 220R -> 1K
- R7: value 220R -> 0.5R
- U2, U3: value DRV8833PWP -> DRV8411PWPR; footprint Package_SO:HTSSOP-16-1EP_4.4x5mm_P0.65mm_EP3.4x5mm_Mask2.46x2.31mm_ThermalVias -> Rocketry_Easyeda:HTSSOP-16_L5.0-W4.4-P0.65-LS6.4-TL-EP-1
- moved C6 113.3 mm to (219.5, 57.1)
- moved Q1 111.4 mm to (244.3, 86.0)
- moved D2 106.7 mm to (223.6, 108.5)
- moved D4 106.7 mm to (237.6, 108.5)
- moved D5 106.7 mm to (230.3, 108.5)
- moved R13 106.7 mm to (237.1, 107.0)
- moved C7 96.4 mm to (205.1, 71.1)
- moved C8 96.4 mm to (209.3, 67.5)
- moved D3 96.4 mm to (215.8, 77.0)
- moved FB1 96.4 mm to (207.1, 69.6)
- moved R12 96.4 mm to (213.8, 72.8)
- moved R2 96.4 mm to (239.0, 61.0)
- moved R3 96.4 mm to (239.0, 66.5)
- moved R4 96.4 mm to (234.8, 91.8)
- moved R5 96.4 mm to (210.3, 72.8)
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Connections:
- net /USB_D+ renamed Net-(U1-PA12)
- C16 pad 1: +3.3V -> /BATT+_IN
- C17 pad 1: -BATT -> /BATT+_IN
- C17 pad 2: +3.3V -> -BATT
- C19 pad 1: -BATT -> /BATT+_IN
- C19 pad 2: +3.3V -> -BATT
- C21 pad 1: /BATT+_IN -> +3.3VA
- C25 pad 1: +5V -> Net-(D1-A)
- C26 pad 1: +5V -> Net-(D1-A)
- C7 pad 1: +3.3V -> +3.3VA
- C8 pad 1: /NRST -> +3.3V
- D1 pad 1: /BATT+_IN -> +5V
- D1 pad 2: VBUS -> Net-(D1-A)
- FB1 pad 1: +3.3VA -> +3.3V
- FB1 pad 2: +3.3V -> +3.3VA
- J2 pad 4: -BATT -> /NRST
- J4 pad 2: /I2C1_SCL -> Net-(J4-Pin_2)
- J4 pad 3: /I2C1_SDA -> +BATT
- L2 pad 2: +5V -> Net-(D1-A)
- R11 pad 1: +5V -> Net-(D1-A)
- R7 pad 1: -BATT -> Net-(U7-VIN)
- R7 pad 2: /POWER_LED_K -> +5V
- U1 pad 18: unconnected-(U1-PB0-Pad18) -> /BUZZER_CTRL
- U1 pad 19: unconnected-(U1-PB1-Pad19) -> /GPIO_EXT1
- U1 pad 2: unconnected-(U1-PC13-Pad2) -> /NSLEEP1
- U1 pad 20: unconnected-(U1-PB2-Pad20) -> /GPIO_EXT2
- U1 pad 21: unconnected-(U1-PB10-Pad21) -> /BAT_STAT
- U1 pad 29: /I2C3_SCL -> unconnected-(U1-PA8-Pad29)
- U1 pad 3: unconnected-(U1-PC14-Pad3) -> /NSLEEP2
- U1 pad 38: unconnected-(U1-PA15-Pad38) -> /SPI1_NSS
- U1 pad 39: unconnected-(U1-PB3-Pad39) -> /SPI1_CLK
- U1 pad 40: /I2C3_SDA -> /SPI1_MISO
- U1 pad 41: unconnected-(U1-PB5-Pad41) -> /SPI1_MOSI
- U1 pad 42: /I2C1_SCL -> unconnected-(U1-PB6-Pad42)
- U1 pad 43: /I2C1_SDA -> unconnected-(U1-PB7-Pad43)
- U2 pad 1: +3.3V -> /NSLEEP1
- U2 pad 11: +3.3V -> unconnected-(U2-NC-Pad11)
- U2 pad 14: +3.3V -> unconnected-(U2-NC-Pad14)
- U2 pad 3: unconnected-(U2-AISEN-Pad3) -> -BATT
- U2 pad 6: unconnected-(U2-BISEN-Pad6) -> -BATT
- U3 pad 1: +3.3V -> /NSLEEP2
- U3 pad 11: +3.3V -> unconnected-(U3-NC-Pad11)
- U3 pad 14: +3.3V -> unconnected-(U3-NC-Pad14)
- U3 pad 3: unconnected-(U3-AISEN-Pad3) -> -BATT
- U3 pad 6: unconnected-(U3-BISEN-Pad6) -> -BATT
- USB2 pad 11: VBUS -> +5V
- USB2 pad 2: VBUS -> +5V
Routing:
- net +3.3V: track 173.0 -> 0.00 mm, vias 19 -> 0
- net -BATT: track 73.4 -> 0.00 mm, vias 27 -> 0
- net /BATT+_IN: track 70.1 -> 0.00 mm, vias 3 -> 0
- net VBUS: track 46.8 -> 0.00 mm
- net +5V: track 40.1 -> 0.00 mm, vias 4 -> 0
- net Net-(U1-PA12): track 26.6 -> 0.00 mm
- net /USB_D-: track 26.6 -> 0.00 mm
- net /TIM3_CH2: track 23.8 -> 0.00 mm
- net /TIM3_CH1: track 22.9 -> 0.00 mm
- net +BATT: track 22.7 -> 0.00 mm
- net /TIM2_CH2: track 21.5 -> 0.00 mm
- net /PI_POWER: track 21.4 -> 0.00 mm, vias 2 -> 0
- net /TIM2_CH1: track 21.3 -> 0.00 mm
- net /TIM2_CH4: track 20.0 -> 0.00 mm
- net /TIM2_CH3: track 19.4 -> 0.00 mm
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- added copper zone on F.Cu, net +BATT
- removed copper zone on B.Cu, net -BATT
- removed copper zone on F.Cu, net -BATT
Other:
- board text removed: "BATT"
- board text removed: "BATT SWITCH"
- board text removed: "BOOT MODE SWITCH"
- board text removed: "POWER"
- board text removed: "RPI POWER"
- board text removed: "RPI POWER SWITCH"
- board text removed: "RPI ZERO 2W CONN"
- board text removed: "STM LED"

Commit message: final V2
Parts:
- removed C20, C21: 100nF, Capacitor_SMD:C_0402_1005Metric
- removed D9: SS34_C8678, Rocketry_Easyeda:SMA_L4.3-W2.6-LS5.2-RD
- removed R24: 5K1, Resistor_SMD:R_0402_1005Metric
- removed U6: LSM6DSL, Package_LGA:LGA-14_3x2.5mm_P0.5mm_LayoutBorder3x4y
- added C36: 100uF, Capacitor_SMD:C_1206_3216Metric, F.Cu at (98.6, 77.3)
- added C37: 100nF, Capacitor_SMD:C_0402_1005Metric, F.Cu at (96.8, 77.4)
- added J8: Conn_01x05_Socket, Connector_JST:JST_XH_S5B-XH-A_1x05_P2.50mm_Horizontal, F.Cu at (120.3, 73.7)
- added U8: RZ7899-MS, Rocketry_Easyeda:SOIC-8_L4.9-W3.9-P1.27-LS6.0-BL, F.Cu at (92.1, 93.7)
- C13: value 100n -> 100nF
- C16, C19: value 10uF -> 100uF; footprint Capacitor_SMD:C_0603_1608Metric -> Capacitor_SMD:C_1206_3216Metric
- D6: value LED -> KT-603R
- R10: value 10K -> 7.5K; footprint Resistor_SMD:R_0402_1005Metric -> Resistor_SMD:R_0603_1608Metric
- R11: value 63.4K -> 47K
- R16: value 91K -> 75K
- R22: footprint Resistor_SMD:R_0402_1005Metric -> Resistor_SMD:R_0603_1608Metric
- R7: value 0.5R -> 1R; footprint Resistor_SMD:R_0402_1005Metric -> Resistor_SMD:R_0603_1608Metric
- U2, U3: value DRV8411PWPR -> RZ7899-MS; footprint Rocketry_Easyeda:HTSSOP-16_L5.0-W4.4-P0.65-LS6.4-TL-EP-1 -> Rocketry_Easyeda:SOIC-8_L4.9-W3.9-P1.27-LS6.0-BL
- moved D7 108.0 mm to (98.2, 71.2), turned to 90 degrees
- moved Q1 107.0 mm to (137.8, 96.2), turned to 0 degrees
- moved D5 102.9 mm to (127.7, 115.3), turned to 0 degrees
- moved C6 98.5 mm to (124.7, 83.8), turned to 90 degrees
- moved R22 98.1 mm to (101.0, 74.0)
- moved R2 97.1 mm to (143.6, 78.8)
- moved R3 96.8 mm to (143.6, 82.7)
- moved D4 94.5 mm to (143.4, 115.3), turned to 180 degrees
- moved R13 94.5 mm to (142.9, 113.8), turned to 0 degrees
- moved R28 92.5 mm to (106.1, 101.1), turned to 180 degrees
- moved C8 91.9 mm to (124.5, 103.1)
- moved D6 90.0 mm to (106.4, 102.5), turned to 180 degrees
- moved FB1 89.1 mm to (123.5, 100.5), turned to 180 degrees
- moved R26 89.0 mm to (109.7, 93.4)
- moved R6 88.8 mm to (124.4, 89.8), turned to 180 degrees
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Connections:
- net Net-(D1-A) renamed /5.55V
- net Net-(U1-PA12) renamed /USB_D+
- C32 pad 1: +5V -> VBUS
- D10 pad 2: +5V -> VBUS
- D12 pad 2: +5V -> VBUS
- J4 pad 1: -BATT -> +BATT
- J4 pad 3: +BATT -> -BATT
- L4 pad 2: +5V -> VBUS
- Q3 pad 1: +5V -> VBUS
- Q5 pad 1: Net-(Q5-G) -> Net-(Q3-D)
- R14 pad 2: +5V -> VBUS
- R23 pad 2: +5V -> VBUS
- R25 pad 1: Net-(Q5-G) -> Net-(Q3-D)
- R26 pad 1: +5V -> VBUS
- R5 pad 2: /ADC1_IN4 -> /ADC1_IN9
- R6 pad 1: /ADC1_IN4 -> /ADC1_IN9
- R7 pad 2: +5V -> VBUS
- U1 pad 14: /ADC1_IN4 -> unconnected-(U1-PA4-Pad14)
- U1 pad 18: /BUZZER_CTRL -> /BAT_STAT
- U1 pad 19: /GPIO_EXT1 -> /ADC1_IN9
- U1 pad 20: /GPIO_EXT2 -> unconnected-(U1-PB2-Pad20)
- U1 pad 21: /BAT_STAT -> unconnected-(U1-PB10-Pad21)
- U1 pad 39: /SPI1_CLK -> unconnected-(U1-PB3-Pad39)
- U1 pad 40: /SPI1_MISO -> unconnected-(U1-PB4-Pad40)
- U1 pad 41: /SPI1_MOSI -> /GPIO_EXT5
- U1 pad 42: unconnected-(U1-PB6-Pad42) -> /I2C1_CLK
- U1 pad 43: unconnected-(U1-PB7-Pad43) -> /I2C1_SDA
- U1 pad 45: unconnected-(U1-PB8-Pad45) -> /BUZZER_CTRL
- U2 pad 1: /NSLEEP1 -> /TIM2_CH4
- U2 pad 2: Net-(J5-Pin_1) -> /TIM2_CH3
- U2 pad 4: Net-(J5-Pin_2) -> /BATT+_IN
- U2 pad 6: -BATT -> Net-(J6-Pin_1)
- U2 pad 8: unconnected-(U2-nFAULT-Pad8) -> Net-(J6-Pin_2)
- U3 pad 1: /NSLEEP2 -> /TIM2_CH2
- U3 pad 2: Net-(J7-Pin_1) -> /TIM2_CH1
- U3 pad 4: Net-(J7-Pin_2) -> /BATT+_IN
- U3 pad 5: unconnected-(U3-BOUT2-Pad5) -> Net-(J5-Pin_1)
- U3 pad 6: -BATT -> Net-(J5-Pin_1)
- U3 pad 7: unconnected-(U3-BOUT1-Pad7) -> Net-(J5-Pin_2)
- U3 pad 8: unconnected-(U3-nFAULT-Pad8) -> Net-(J5-Pin_2)
- USB2 pad 11: +5V -> VBUS
- USB2 pad 2: +5V -> VBUS
Routing:
- net +3.3V: track 0.00 -> 130.1 mm, vias 0 -> 7
- net VBUS: track 0.00 -> 81.1 mm, vias 0 -> 21
- net /BATT+_IN: track 0.00 -> 64.6 mm, vias 0 -> 31
- net /TIM3_CH2: track 0.00 -> 42.9 mm
- net /TIM3_CH1: track 0.00 -> 42.6 mm
- net /TIM2_CH1: track 0.00 -> 36.2 mm
- net /TIM2_CH2: track 0.00 -> 35.9 mm
- net /TIM2_CH4: track 0.00 -> 35.5 mm
- net /TIM2_CH3: track 0.00 -> 35.2 mm
- net /BOOT0: track 0.00 -> 32.2 mm
- net /BUZZER_CTRL: track 0.00 -> 31.3 mm
- net +BATT: track 0.00 -> 30.5 mm, vias 0 -> 3
- net /PI_POWER: track 0.00 -> 24.6 mm
- net /USART1_TX: track 0.00 -> 22.7 mm
- net +3.3VA: track 0.00 -> 22.4 mm, vias 0 -> 2
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- added copper zone on F.Cu, net +3.3VA
- added copper zone on B.Cu, net +BATT
- added copper zone on B.Cu, net -BATT
- added copper zone on F.Cu, net -BATT
- added copper zone on F.Cu, net /5.55V
- added copper zone on B.Cu, net /BATT+_IN
- added copper zone on F.Cu, net Net-(C31-Pad2)
- added copper zone on F.Cu, net Net-(J5-Pin_1)
- added copper zone on F.Cu, net Net-(J5-Pin_2)
- added copper zone on F.Cu, net Net-(J6-Pin_1)
- added copper zone on F.Cu, net Net-(J6-Pin_2)
- added copper zone on F.Cu, net Net-(J7-Pin_1)
- added copper zone on F.Cu, net Net-(J7-Pin_2)
- added copper zone on B.Cu, net VBUS
- added copper zone on F.Cu, net VBUS
- removed copper zone on F.Cu, net +5V
Other:
- board text added: "BATT"
- board text added: "BATT (O/I)"
- board text added: "BATT CHRG"
- board text added: "BOOT0 (I/O)"
- board text added: "DEBUG LED"
- board text added: "IMU"
- board text added: "PWR"
- board text added: "RPI"
- board text added: "RPI CONN"
- board text added: "RPI POWER SWITCH (I/O)"
- board text added: "SWD"
- board text removed: "IMU CONN"
- board text removed: "SERIAL DEBUG"
