File: Electrical/VolleyBot.kicad_sch (KiCad schematic)
At the start: 66 parts, among them J1 Conn_01x04_Pin, J2 Conn_01x04_Pin, J3 Conn_01x02_Pin, J4 Conn_01x04_Socket, J5 Conn_01x02_Socket, J6 Conn_01x02_Socket, J7 Conn_01x02_Socket, SW1 SW_SPDT, U1 STM32F411CEU6, U2 DRV8833PWP, U3 DRV8833PWP, U4 AP62300TWU, U5 AP62300TWU, Y1 16MHz

Commit message: routed pcb
Parts:
- J3: footprint TerminalBlock:TerminalBlock_MaiXu_MX126-5.0-02P_1x02_P5.00mm -> Rocketry_Manual:Screw_Terminal_2_Pins
Connections:
- net VBATT is gone; now on net +BATT: C18.1, C21.1, U2.12 (VM), U3.12 (VM)
Changed lines of the file:
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@@
 		)
 	)
-	(label "VBATT"
-		(at 257.81 147.955 0)
-		(effects
-			(font
-				(size 1.27 1.27)
-			)
-			(justify left bottom)
-		)
-	)
 	(label "BOOT0"
 		(at 102.87 62.23 0)
@@
 		)
 	)
-	(label "VBATT"
-		(at 262.255 212.09 0)
-		(effects
-			(font
-				(size 1.27 1.27)
-			)
-			(justify left bottom)
-		)
-	)
 	(label "USART1_RX"
 		(at 146.05 82.55 0)
@@
 			)
 		)
-		(property "Footprint" "TerminalBlock:TerminalBlock_MaiXu_MX126-5.0-02P_1x02_P5.00mm"
+		(property "Footprint" "Rocketry_Manual:Screw_Terminal_2_Pins"
 			(at 72.39 200.66 0)
 			(effects
@@
 	)
 	(symbol
+		(lib_id "power:+BATT")
+		(at 262.255 212.09 0)
+		(unit 1)
+		(exclude_from_sim no)
+		(in_bom yes)
+		(on_board yes)
+		(dnp no)
+		(property "Reference" "#PWR048"
+			(at 262.255 215.9 0)
+			(effects
+				(font
+					(size 1.27 1.27)
+				)
+				(hide yes)
+			)
+		)
+		(property "Value" "+BATT"
+			(at 262.255 207.01 0)
+			(effects
+				(font
+					(size 1.27 1.27)
+				)
+			)
+		)
+		(property "Footprint" ""
+			(at 262.255 212.09 0)
+			(effects
+				(font
+					(size 1.27 1.27)
+				)
+				(hide yes)
+			)
+		)
+		(property "Datasheet" ""
+			(at 262.255 212.09 0)
+			(effects
+				(font
+					(size 1.27 1.27)
+				)
+				(hide yes)
+			)
+		)
+		(property "Description" "Power symbol creates a global label with name \"+BATT\""
+			(at 262.255 212.09 0)
+			(effects
+				(font
+					(size 1.27 1.27)
+				)
+				(hide yes)
+			)
+		)
+		(pin "1"
+		)
+		(instances
+			(project "VolleyBot"
+				(path "/ccc4a57f-b426-4aed-bfc6-2903311eec96"
+					(reference "#PWR048")
+					(unit 1)
+				)
+			)
+		)
+	)
+	(symbol
 		(lib_id "Mechanical:MountingHole")
 		(at 208.915 33.655 0)
@@
 					(unit 1)
 				)
+			)
+		)
+	)
+	(symbol
+		(lib_id "power:+BATT")
+		(at 257.81 147.955 0)
+		(unit 1)
+		(exclude_from_sim no)
+		(in_bom yes)
+		(on_board yes)
+		(dnp no)
+		(property "Reference" "#PWR011"
+			(at 257.81 151.765 0)
+			(effects
+				(font
+					(size 1.27 1.27)
+				)
+				(hide yes)
+			)
+		)
+		(property "Value" "+BATT"
+			(at 257.81 142.875 0)
+			(effects
+				(font
+					(size 1.27 1.27)
+				)
+			)
+		)
+		(property "Footprint" ""
+			(at 257.81 147.955 0)
+			(effects
+				(font
+					(size 1.27 1.27)
+				)
+				(hide yes)
+			)
+		)
+		(property "Datasheet" ""
+			(at 257.81 147.955 0)
+			(effects
+				(font
+					(size 1.27 1.27)
+				)
+				(hide yes)
+			)
+		)
+		(property "Description" "Power symbol creates a global label with name \"+BATT\""
+			(at 257.81 147.955 0)
+			(effects
+				(font
+					(size 1.27 1.27)
+				)
+				(hide yes)
+			)
+		)
+		(pin "1"
+		)
+		(instances
+			(project "VolleyBot"
+				(path "/ccc4a57f-b426-4aed-bfc6-2903311eec96"
+					(reference "#PWR011")
+					(unit 1)
+				)

Commit message: pcb made
Parts:
- removed J3: Conn_01x02_Pin, Rocketry_Manual:Screw_Terminal_2_Pins, symbol Connector:Conn_01x02_Pin
- added C27: 10uF, Capacitor_SMD:C_0603_1608Metric, symbol Device:C
- added C28, C29: 10u, Capacitor_SMD:C_0603_1608Metric, symbol Device:C
- added C30: 47uF, Capacitor_SMD:C_0805_2012Metric, symbol Device:C
- added C31: 4.7uF, Capacitor_SMD:C_0603_1608Metric, symbol Device:C
- added C32: 44uF, Capacitor_SMD:C_0805_2012Metric, symbol Device:C
- added D4, D5: LED, LED_SMD:LED_0603_1608Metric, symbol Device:LED
- added J3: Conn_01x02_Socket, Connector_AMASS:AMASS_XT60PW-F_1x02_P7.20mm_Horizontal, symbol Connector:Conn_01x02_Socket
- added J8: Conn_01x03_Socket, Connector_JST:JST_XH_S3B-XH-A_1x03_P2.50mm_Horizontal, symbol Connector:Conn_01x03_Socket
- added L3: 1uH, Inductor_SMD:L_0603_1608Metric, symbol Device:L
- added Q1, Q2: AO3401A, Rocketry_Easyeda:SOT-23_L2.9-W1.3-P1.90-LS2.4-BR, symbol Rocketry_Easyeda:AO3401A
- added R13, R20: 220R, Resistor_SMD:R_0402_1005Metric, symbol Device:R
- added R14, R16, R19, R4: 10K, Resistor_SMD:R_0402_1005Metric, symbol Device:R
- added R15: 75R, Resistor_SMD:R_0402_1005Metric, symbol Device:R
- added R17: 300R, Resistor_SMD:R_0402_1005Metric, symbol Device:R
- added R18: 1K, Resistor_SMD:R_0402_1005Metric, symbol Device:R
- added SW2, SW3: SW_SPDT, Button_Switch_SMD:SW_SPDT_PCM12, symbol Switch:SW_SPDT
- added U6: BQ25887, Package_DFN_QFN:VQFN-24-1EP_4x4mm_P0.5mm_EP2.5x2.5mm, symbol Battery_Management:BQ25887
- C1, C12, C18, C21, C23: value 10u -> 10uF
- C10, C9: value 10p -> 10pF
- C14, C15, C25, C26: value 22u -> 22uF
- C17, C19: value 10n -> 10nF
- C2, C22, C24, C3, C4, C8: value 100n -> 100nF
- C5: value 10n -> 100nF
- C6, C7: value 1u -> 1uF
- FB1: value 120R -> 600R
- R5: value 6K8 -> 15K
Connections:
- net +5V: now also Q1.1 (G), Q1.2 (S), R4.2; no longer J1.4 (Pin_4)
- net +BATT: now also C29.2, J3.1 (Pin_1), J8.1 (Pin_1), Q2.1 (G), Q2.2 (S), R19.2, U6.13 (BAT), U6.14 (BAT); no longer C12.1, C18.1, C21.1, C23.1, D1.1 (K), R5.1, U2.12 (VM), U3.12 (VM), U4.3 (IN), U5.3 (IN)
- net -BATT: now also C27.1, C28.1, C29.1, C31.2, C32.2, J3.2 (Pin_2), J8.3 (Pin_3), R13.1, R14.2, R18.2, R20.1, SW2.2 (B), SW3.2 (B), U6.19 (GND), U6.20 (GND)
- net VBUS: now also C27.2, R16.1, U6.23 (VBUS), U6.24 (PSEL)
- net I2C1_SCL: now reaches J4.2 (Pin_2), U1.42 (PB6)
- net I2C1_SDA: now reaches J4.3 (Pin_3), U1.43 (PB7)
- net I2C3_SCL: now reaches U1.29 (PA8)
- net I2C3_SCL: now also U6.5 (SCL)
- net I2C3_SDA: now reaches U1.40 (PB4)
- net I2C3_SDA: now also U6.4 (SDA)
- new net: C30.1, L3.2, U6.17 (SW), U6.18 (SW)
- new net: C30.2, U6.12 (BTST)
- new net: D4.1 (K), R13.2
- new net: R4.1, SW2.1 (A)
- new net: D5.1 (K), R20.2
- new net: C28.2, L3.1, U6.21 (PMID), U6.22 (PMID)
- new net: R15.1, U6.10 (CBSET)
- new net: R14.1, U6.1 (~{PG})
- new net: C31.1, U6.11 (REGN)
- new net: C32.1, U6.15 (SNS), U6.16 (SNS)
- new net: R16.2, U6.6 (~{INT})
- new net: R18.1, U6.8 (ILIM)
- new net: R17.1, U6.9 (MID)
- new net: R19.1, SW3.1 (A)
- new net BATT+_IN: C12.1, C18.1, C21.1, C23.1, D1.1 (K), D5.2 (A), Q2.3 (D), R5.1, U2.12 (VM), U3.12 (VM), U4.3 (IN), U5.3 (IN)
- new net BATT_BALL_MID: J8.2 (Pin_2), R15.2, R17.2
- new net CD_PIN: U6.3 (CD)
- new net PI_POWER: D4.2 (A), J1.4 (Pin_4), Q1.3 (D)
Other:
- note added: "Balance Charger"
- note added: "Battery Shutoff"
- note added: "RPI Power Management"
- moved on the sheet: J7

Commit message: correction of manufacturing files
Parts:
- removed R19: 10K, Resistor_SMD:R_0402_1005Metric, symbol Device:R
- added R21: 10K, Resistor_SMD:R_0402_1005Metric, symbol Device:R
- R11: footprint Resistor_SMD:R_0402_1005Metric -> Resistor_SMD:R_0603_1608Metric
Connections:
- net +5V: now also SW2.1 (A); no longer Q1.1 (G), R4.2
- net +BATT: now also SW3.1 (A); no longer Q2.1 (G)
- net -BATT: now also SW2.3 (C), SW3.3 (C); no longer SW2.2 (B), SW3.2 (B)
- net at R4.1: now also SW2.2 (B); no longer SW2.1 (A)
- new net: R21.1, SW3.2 (B)
- new net: Q2.1 (G), R21.2
- new net: Q1.1 (G), R4.2
Other:
- moved on the sheet: SW2, SW3

Commit message: update
Parts:
- removed C27: 10uF, Capacitor_SMD:C_0603_1608Metric, symbol Device:C
- removed C28, C29: 10u, Capacitor_SMD:C_0603_1608Metric, symbol Device:C
- removed C30: 47uF, Capacitor_SMD:C_0805_2012Metric, symbol Device:C
- removed C31: 4.7uF, Capacitor_SMD:C_0603_1608Metric, symbol Device:C
- removed C32: 44uF, Capacitor_SMD:C_0805_2012Metric, symbol Device:C
- removed J2: Conn_01x04_Pin, Connector_PinHeader_2.54mm:PinHeader_1x04_P2.54mm_Horizontal, symbol Connector:Conn_01x04_Pin
- removed J4: Conn_01x04_Socket, Connector_JST:JST_XH_S4B-XH-A_1x04_P2.50mm_Horizontal, symbol Connector:Conn_01x04_Socket
- removed J8: Conn_01x03_Socket, Connector_JST:JST_XH_S3B-XH-A_1x03_P2.50mm_Horizontal, symbol Connector:Conn_01x03_Socket
- removed L3: 1uH, Inductor_SMD:L_0603_1608Metric, symbol Device:L
- removed R14, R16: 10K, Resistor_SMD:R_0402_1005Metric, symbol Device:R
- removed R15: 75R, Resistor_SMD:R_0402_1005Metric, symbol Device:R
- removed R17: 300R, Resistor_SMD:R_0402_1005Metric, symbol Device:R
- removed R18: 1K, Resistor_SMD:R_0402_1005Metric, symbol Device:R
- removed U2, U3: DRV8833PWP, Package_SO:HTSSOP-16-1EP_4.4x5mm_P0.65mm_EP3.4x5mm_Mask2.46x2.31mm_ThermalVias, symbol Driver_Motor:DRV8833PWP
- removed U6: BQ25887, Package_DFN_QFN:VQFN-24-1EP_4x4mm_P0.5mm_EP2.5x2.5mm, symbol Battery_Management:BQ25887
- added J2: Conn_01x05_Socket, Connector_JST:JST_XH_S5B-XH-A_1x05_P2.50mm_Horizontal, symbol Connector:Conn_01x05_Socket
- added U2, U3: DRV8411PWPR, Rocketry_Easyeda:HTSSOP-16_L5.0-W4.4-P0.65-LS6.4-TL-EP-1, symbol ROCKETRY_EASYEDA:DRV8411PWPR
- added U6: LSM6DSL, Package_LGA:LGA-14_3x2.5mm_P0.5mm_LayoutBorder3x4y, symbol Sensor_Motion:LSM6DSL
- added U7: IP2326, Rocketry_Easyeda:VQFN-24_L4.0-W4.0-P0.50-BL-EP2.5, symbol ROCKETRY_EASYEDA:IP2326
- C16: value 2.2uF -> 10uF; footprint Capacitor_SMD:C_0402_1005Metric -> Capacitor_SMD:C_0603_1608Metric
- C17: value 10nF -> 100nF
- C18: value 10uF -> 100nF; footprint Capacitor_SMD:C_0603_1608Metric -> Capacitor_SMD:C_0402_1005Metric
- C19: value 10nF -> 10uF; footprint Capacitor_SMD:C_0402_1005Metric -> Capacitor_SMD:C_0603_1608Metric
- C20: value 2.2uF -> 100nF; footprint Capacitor_SMD:C_0402_1005Metric -> (none)
- C21: value 10uF -> 100nF; footprint Capacitor_SMD:C_0603_1608Metric -> (none)
- C6: value 1uF -> 10uF; footprint Capacitor_SMD:C_0402_1005Metric -> Capacitor_SMD:C_0603_1608Metric
- C7: value 1uF -> 10uF; footprint Capacitor_SMD:C_0402_1005Metric -> Capacitor_SMD:C_0805_2012Metric
- C8: value 100nF -> 10uF; footprint Capacitor_SMD:C_0402_1005Metric -> Capacitor_SMD:C_0805_2012Metric
- FB1: value 600R -> 100R@100MHz; footprint Inductor_SMD:L_0603_1608Metric -> (none)
- J5, J6, J7: footprint Connector_JST:JST_XH_S2B-XH-A_1x02_P2.50mm_Horizontal -> Connector_JST:JST_XH_B2B-XH-A_1x02_P2.50mm_Vertical
Connections:
- net +3.3V: now also C8.1, FB1.1, J2.1 (Pin_1), U6.8 (VDD); no longer C16.1, C17.2, C19.2, C7.1, FB1.2
- net +3.3VA: now also C21.1, C7.1, FB1.2, U6.5 (VDDIO); no longer FB1.1
- net +BATT: now also C16.1, C17.1, C18.1, C19.1, U2.12 (VM), U3.12 (VM)
- net -BATT: now also C17.2, C19.2, J2.5 (Pin_5), U2.13 (GND), U2.17 (EP), U2.3 (AISEN), U2.6 (BISEN), U3.13 (GND), U3.17 (EP), U3.3 (AISEN), U3.6 (BISEN), U6.2 (SDX), U6.3 (SCX), U6.6 (GND), U6.7 (GND); no longer C17.1, C19.1
- net BATT+_IN: no longer C18.1, C21.1
- net NRST: now also J2.4 (Pin_4); no longer C8.1
- net SWCLK: now also J2.2 (Pin_2)
- net SWDIO: now also J2.3 (Pin_3)
- net TIM2_CH1: now also U2.16 (AIN1)
- net TIM2_CH2: now also U2.15 (AIN2)
- net TIM2_CH3: now also U2.10 (BIN2)
- net TIM2_CH4: now also U2.9 (BIN1)
- net TIM3_CH1: now also U3.16 (AIN1)
- net TIM3_CH2: now also U3.15 (AIN2)
- net at J5.1 (Pin_1): now also U2.4 (AOUT2)
- net at J5.2 (Pin_2): now also U2.2 (AOUT1)
- net at J6.1 (Pin_1): now also U2.7 (BOUT1)
- net at J6.2 (Pin_2): now also U2.5 (BOUT2)
- net at J7.1 (Pin_1): now also U3.4 (AOUT2)
- net at J7.2 (Pin_2): now also U3.2 (AOUT1)
- net GPIO_EXT1: now reaches U1.19 (PB1)
- net GPIO_EXT1: now also U6.4 (INT1)
- net GPIO_EXT2: now reaches U1.20 (PB2)
- net GPIO_EXT2: now also U6.9 (INT2)
- net NSLEEP2: now reaches U1.3 (PC14)
- net NSLEEP2: now also U3.1 (nSLEEP)
- net SPI1_NSS: now reaches U1.38 (PA15)
- net SPI1_NSS: now also U6.12 (CS)
- net SPI1_CLK: now reaches U1.39 (PB3)
- net SPI1_CLK: now also U6.13 (SCL)
- net NSLEEP1: now reaches U1.4 (PC15)
- net NSLEEP1: now also U2.1 (nSLEEP)
- net SPI1_MOSI: now reaches U1.41 (PB5)
- net SPI1_MOSI: now also U6.14 (SDA)
- net I2C1_SCL: no longer names the net of U1.42 (PB6)
- net I2C1_SDA: no longer names the net of U1.43 (PB7)
- net I2C3_SCL: no longer names the net of U1.29 (PA8)
- net I2C3_SDA renamed SPI1_MISO
- net SPI1_MISO: now also U6.1 (SDO/SA0)
- no-connect marks 0 -> 6
Other:
- note added: "IMU"
- note removed: "Balance Charger"
- moved on the sheet: C12, C13, C14, C15, D1, D2, L1, R7, R8, R9, U4

Commit message: bat charge
Parts:
- added C27, C28, C32, C33: 10uF, symbol Device:C
- added C29, C30: 22uF, symbol Device:C
- added C31: 100nF, symbol Device:C
- added D6: LED, symbol Device:LED
- added J4: Conn_01x03_Socket, symbol Connector:Conn_01x03_Socket
- added L3: FNR6045S2R2MT, symbol Device:L
- added R14: 5K1, symbol Device:R
- added R15: 220R, symbol Device:R
- R7: value 220R -> 0.5R; footprint Resistor_SMD:R_0402_1005Metric -> (none)
Connections:
- net -BATT: now also U7.18 (PGND), U7.24 (VBAT_GND), U7.25 (EP), C27.2, C28.2, C29.2, C30.2, C32.2, C33.2, D6.1 (K), J4.1 (Pin_1), R14.1; no longer C10.2, C9.2, R7.1
- net POWER_LED_K: no longer R7.2
- net VBUS: now also R7.2, C32.1, L3.2, R14.2
- net BAT_EN: now reaches U7.12 (EN)
- net at U7.13 (VIN): now also R7.1, C33.1
- net at U7.14 (BST): now also C31.1
- net at U7.15 (LX): now also U7.16 (LX), U7.17 (LX), C31.2, L3.1
- net at U7.19 (VSYS): now also U7.20 (VSYS), C29.1, C30.1
- net at U7.21 (VOUT): now also U7.22 (VOUT), C27.1, C28.1, J4.3 (Pin_3)
- net at U7.23 (VBATM): now also J4.2 (Pin_2)
- net BAT_STAT: now reaches U7.5 (BAT_STAT)
- net at U7.6 (LED): now also R15.2
- net USB_D+: no longer names the net of U1.33 (PA12), USB2.6 (DP1), USB2.8 (DP2)
- new net: D6.2 (A), R15.1
- new net GND2: C10.2, C9.2
- no-connect marks 6 -> 8
Other:
- moved on the sheet: U7, Y1

Commit message: schem done
Parts:
- removed D1: 1N5819WS, Diode_SMD:D_SOD-323, symbol Diode:1N5819WS
- removed L3: FNR6045S2R2MT, symbol Device:L
- removed R20: 220R, Resistor_SMD:R_0402_1005Metric, symbol Device:R
- added BUZZER1: FUET-8530H-3.6V, Rocketry_Easyeda:BUZ-SMD_4P-L8.5-W8.5_FUET-8530-05, symbol Rocketry_Easyeda:FUET-8530H-3.6V
- added C34, C35: 100nF, Capacitor_SMD:C_0402_1005Metric, symbol Device:C
- added D1, D10, D12, D9: SS34_C8678, Rocketry_Easyeda:SMA_L4.3-W2.6-LS5.2-RD, symbol Rocketry_Easyeda:SS34_C8678
- added D7, D8: 1N5819WS, Diode_SMD:D_SOD-323, symbol Diode:1N5819WS
- added L4: FNR6045S2R2MT, Rocketry_Easyeda:IND-SMD_L6.0-W6.0_FNR60XXS, symbol Rocketry_Easyeda:FNR6045S2R2MT
- added Q3: AO3400A, Rocketry_Easyeda:SOT-23-3_L2.9-W1.3-P1.90-LS2.4-BR, symbol Rocketry_Easyeda:AO3400A
- added Q4: SS8050, Package_TO_SOT_SMD:SOT-23, symbol Transistor_BJT:SS8050
- added Q5: AO3401A, Rocketry_Easyeda:SOT-23_L2.9-W1.3-P1.90-LS2.4-BR, symbol Rocketry_Easyeda:AO3401A
- added R16: 91K, Resistor_SMD:R_0603_1608Metric, symbol Device:R
- added R17: 120K, Resistor_SMD:R_0603_1608Metric, symbol Device:R
- added R18: 51K, Resistor_SMD:R_0603_1608Metric, symbol Device:R
- added R19: 100R, Resistor_SMD:R_1206_3216Metric, symbol Device:R
- added R22: 680R, Resistor_SMD:R_0402_1005Metric, symbol Device:R
- added R23, R26: 10K, Resistor_SMD:R_0402_1005Metric, symbol Device:R
- added R24: 5K1, Resistor_SMD:R_0402_1005Metric, symbol Device:R
- added R25: 100K, Resistor_SMD:R_0603_1608Metric, symbol Device:R
- added R27, R28: 1K, Resistor_SMD:R_0402_1005Metric, symbol Device:R
- C20, C21, C31: footprint (none) -> Capacitor_SMD:C_0402_1005Metric
- C27, C28, C32, C33: footprint (none) -> Capacitor_SMD:C_0603_1608Metric
- C29, C30: footprint (none) -> Capacitor_SMD:C_0805_2012Metric
- D6: footprint (none) -> LED_SMD:LED_0603_1608Metric
- FB1: value 100R@100MHz -> C14709; footprint (none) -> Inductor_SMD:L_0603_1608Metric
- J4: footprint (none) -> Connector_JST:JST_XH_S3B-XH-A_1x03_P2.50mm_Horizontal
- J5, J6, J7: footprint Connector_JST:JST_XH_B2B-XH-A_1x02_P2.50mm_Vertical -> Connector_JST:JST_XH_S2B-XH-A_1x02_P2.50mm_Horizontal
- R11: value 56K -> 63.4K
- R12, R13: value 220R -> 1K
- R14, R7: footprint (none) -> Resistor_SMD:R_0402_1005Metric
- R15: value 220R -> 1K; footprint (none) -> Resistor_SMD:R_0402_1005Metric
Connections:
- net GND2 is gone; now on net -BATT: C10.2, C9.2
- net VBUS is gone; now on net +5V: C32.1, R14.2, R7.2, USB2.11 (VBUS), USB2.2 (VBUS)
- net +3.3V: now also BUZZER1.1, D7.1 (K)
- net +5V: now also D1.1 (K), D10.2 (A), D12.2 (A), D9.2 (A), L4.2, Q3.1 (G), R23.2, R26.1; no longer C25.1, C26.1, L2.2, R11.1
- net +BATT: now also C27.1, C28.1, J4.3 (Pin_3), U7.21 (VOUT), U7.22 (VOUT), C34.1, C35.1, Q5.2 (S), R24.2, R25.2; no longer C16.1, C17.1, C18.1, C19.1, U2.12 (VM), U3.12 (VM)
- net -BATT: now also R15.1, BUZZER1.3, BUZZER1.4, C34.2, D8.1 (K), Q3.2 (S), Q4.2 (E), R16.1, R17.1, R18.1, R27.2
- net BATT+_IN: now also C16.1, C17.1, C18.1, C19.1, U2.12 (VM), U3.12 (VM), D10.1 (K), D12.1 (K), D9.1 (K)
- net BAT_STAT: now also U1.21 (PB10)
- net NSLEEP1: now also U1.2 (PC13); no longer U1.4 (PC15)
- net POWER_LED_K: now also R27.1
- net at U2.2 (AOUT1): now also J5.1 (Pin_1); no longer J5.2 (Pin_2)
- net at U2.4 (AOUT2): now also J5.2 (Pin_2); no longer J5.1 (Pin_1)
- net at U2.5 (BOUT2): now also J6.1 (Pin_1); no longer J6.2 (Pin_2)
- net at U2.7 (BOUT1): now also J6.2 (Pin_2); no longer J6.1 (Pin_1)
- net at D5.1 (K): now also R15.2
- net at J4.2 (Pin_2): now also C35.2, R19.2; no longer U7.23 (VBATM)
- net at D6.2 (A): now also R28.2; no longer R15.1
- net BUZZER_CTRL: now reaches U1.18 (PB0)
- net BUZZER_CTRL: now also R22.2
- net at U7.11 (ISET): now also R16.2
- net at C31.2, U7.15 (LX), U7.16 (LX)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: now also L4.1
- net at U7.4 (NTC): now also R18.2
- net at U7.6 (LED): now also R28.1; no longer R15.2
- net at U7.8 (VIN_UVSET): now also R17.2
- net at U3.2 (AOUT1): now also J7.1 (Pin_1); no longer J7.2 (Pin_2)
- net at U3.4 (AOUT2): now also J7.2 (Pin_2); no longer J7.1 (Pin_1)
- net at Q2.1 (G), R21.2: now also Q5.3 (D)
- net BAT_EN: no longer names the net of U7.12 (EN)
- net BAT_EN: now also R26.2
- new net: C25.1, C26.1, D1.2 (A), L2.2, R11.1
- new net: Q4.1 (B), R22.1
- new net: BUZZER1.2, D7.2 (A), Q4.3 (C)
- new net: R19.1, U7.23 (VBATM)
- new net: Q5.1 (G), R25.1
- new net: D8.2 (A), R23.1
- new net: Q3.3 (D), R24.1
- no-connect marks 8 -> 12
Other:
- note added: "BUZZER"
- note added: "Battery Charger"
- moved on the sheet: C16, C17, C18, C19, C27, C28, C29, C30, C31, C32, C33, D5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

Commit message: final V2
Parts:
- removed D9: SS34_C8678, Rocketry_Easyeda:SMA_L4.3-W2.6-LS5.2-RD, symbol Rocketry_Easyeda:SS34_C8678
- removed R24: 5K1, Resistor_SMD:R_0402_1005Metric, symbol Device:R
- removed U2, U3: DRV8411PWPR, Rocketry_Easyeda:HTSSOP-16_L5.0-W4.4-P0.65-LS6.4-TL-EP-1, symbol ROCKETRY_EASYEDA:DRV8411PWPR
- added C36: 100uF, Capacitor_SMD:C_1206_3216Metric, symbol Device:C
- added C37: 100nF, Capacitor_SMD:C_0402_1005Metric, symbol Device:C
- added J8: Conn_01x05_Socket, Connector_JST:JST_XH_S5B-XH-A_1x05_P2.50mm_Horizontal, symbol Connector:Conn_01x05_Socket
- added U2, U3, U8: RZ7899-MS, Rocketry_Easyeda:SOIC-8_L4.9-W3.9-P1.27-LS6.0-BL, symbol Rocketry_Easyeda:RZ7899-MS
- C13: value 100n -> 100nF
- C16, C19: value 10uF -> 100uF; footprint Capacitor_SMD:C_0603_1608Metric -> Capacitor_SMD:C_1206_3216Metric
- C20, C21, U6: now not fitted; now left out of the parts list
- D6: value LED -> KT-603R
- R10: value 10K -> 7.5K; footprint Resistor_SMD:R_0402_1005Metric -> Resistor_SMD:R_0603_1608Metric
- R11: value 63.4K -> 47K
- R16: value 91K -> 75K
- R22: footprint Resistor_SMD:R_0402_1005Metric -> Resistor_SMD:R_0603_1608Metric
- R7: value 0.5R -> 1R; footprint Resistor_SMD:R_0402_1005Metric -> Resistor_SMD:R_0603_1608Metric
Connections:
- net +3.3V: now also J8.5 (Pin_5)
- net +5V: no longer C32.1, D10.2 (A), D12.2 (A), L4.2, Q3.1 (G), R14.2, R23.2, R26.1, R7.2, USB2.11 (VBUS), USB2.2 (VBUS)
- net +BATT: now also J4.1 (Pin_1); no longer J4.3 (Pin_3)
- net -BATT: now also J4.3 (Pin_3), C36.2, C37.2, J8.4 (Pin_4), U2.3 (GND), U3.3 (GND), U8.3 (GND); no longer J4.1 (Pin_1)
- net BATT+_IN: now also C36.1, C37.1, U2.4 (VCC), U3.4 (VCC), U8.4 (VCC)
- net BAT_STAT: now also U1.18 (PB0); no longer U1.21 (PB10)
- net BUZZER_CTRL: now also U1.45 (PB8); no longer U1.18 (PB0)
- net SPI1_CLK: no longer U1.39 (PB3)
- net SPI1_MISO: no longer U1.40 (PB4)
- net SPI1_MOSI: no longer U1.41 (PB5)
- net TIM2_CH1: now also U3.2 (FI)
- net TIM2_CH2: now also U3.1 (BI)
- net TIM2_CH3: now also U2.2 (FI)
- net TIM2_CH4: now also U2.1 (BI)
- net TIM3_CH1: now also U8.2 (FI)
- net TIM3_CH2: now also U8.1 (BI)
- net 5.55V: now reaches C25.1, C26.1, D1.2 (A), L2.2, R11.1
- net at J5.1 (Pin_1): now also U3.5 (FO), U3.6 (FO)
- net at J5.2 (Pin_2): now also U3.7 (BO), U3.8 (BO)
- net at J6.1 (Pin_1): now also U2.5 (FO), U2.6 (FO)
- net at J6.2 (Pin_2): now also U2.7 (BO), U2.8 (BO)
- net USB_D+: now reaches U1.33 (PA12), USB2.6 (DP1), USB2.8 (DP2)
- net I2C1_CLK: now reaches U1.42 (PB6)
- net I2C1_CLK: now also J8.2 (Pin_2)
- net I2C1_SDA: now reaches U1.43 (PB7)
- net I2C1_SDA: now also J8.3 (Pin_3)
- net at Q5.1 (G), R25.1: now also Q3.3 (D)
- net at J7.1 (Pin_1): now also U8.5 (FO), U8.6 (FO)
- net at J7.2 (Pin_2): now also U8.7 (BO), U8.8 (BO)
- net ADC1_IN4 renamed ADC1_IN9
- net ADC1_IN9: now also U1.19 (PB1); no longer U1.14 (PA4)
- net GPIO_EXT1 renamed GPIO_EXT7
- net GPIO_EXT7: no longer U1.19 (PB1)
- net GPIO_EXT2: no longer names the net of U1.20 (PB2)
- net GPIO_EXT2: no longer U6.9 (INT2)
- new net GPIO_EXT5: J8.1 (Pin_1), U1.41 (PB5)
- new net GPIO_EXT6: U6.9 (INT2)
- new net VBUS: C32.1, D10.2 (A), D12.2 (A), L4.2, Q3.1 (G), R14.2, R23.2, R26.1, R7.2, USB2.11 (VBUS), USB2.2 (VBUS)
- no-connect marks 12 -> 6
Other:
- note added: "External IMU (GY-521)"
- note added: "Unused IMU Pins"
- moved on the sheet: BUZZER1, C18, C19, D5, D7, D8, J3, J7, Q2, Q3, Q4, Q5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
